Commit message: add function to get data from gazebo model state

File: urdf/holo.urdf.xacro (robot description, xacro)
@@ -25,5 +25,5 @@
       </geometry>
       <material name = "white"/>
-      <origin xyz = "0 0 0" rpy = "0 0 ${pi/4}"/>
+      <origin xyz = "0 0 0" rpy = "0 0 ${-pi/4}"/>
     </visual>
     <collision>
@@ -31,5 +31,5 @@
         <box size = "${base_side_length} ${base_side_length} 0.2"/>
       </geometry>
-      <origin xyz = "0 0 0" rpy = "0 0 ${pi/4}"/>
+      <origin xyz = "0 0 0" rpy = "0 0 ${-pi/4}"/>
     </collision>
     <xacro:default_inertial mass="8"/>
